Commit message: cleanup: add .gitignore, remove build artifacts, add camera+lidar sensors
- Add .gitignore to exclude build/, install/, log/
- Remove tracked build artifacts from git (2310+ files)
- Add camera.xacro and lidar.xacro as reusable sensor macros
- Fix package.xml dependencies (add ros_gz_bridge, remove unused)
- Add use_sim_time to all ROS nodes for simulation clock sync
- Fix DiffDrive frame_id/child_frame_id for unified TF tree
- Add static TF publisher for LiDAR sensor frame
- Simplify setup.py glob pattern for xacro files

Co-Authored-By: Claude Opus 4.7 <noreply@anthropic.com>

File: src/my_robot/urdf/my_robot.urdf.xacro (robot description, xacro)
@@ -1,4 +1,6 @@
 <?xml version="1.0"?>
 <robot name="my_robot" xmlns:xacro="http://www.ros.org/wiki/xacro">
+  <xacro:include filename="$(find my_robot)/urdf/camera.xacro" />
+  <xacro:include filename="$(find my_robot)/urdf/lidar.xacro" />
   <xacro:property name="M_PI" value="3.1415926"/>
   <xacro:property name="base_mass"   value="2.0" />
@@ -15,4 +17,9 @@
     <color rgba="0.1 0.1 0.1 1.0"/>
   </material>
+  <material name="black">
+    <color rgba="0 0 0 1.0"/>
+  </material>
+  <xacro:camera/>
+  <xacro:rplidar/>
   <!-- 底盘 -->
   <link name="base_link">
@@ -99,4 +106,11 @@
       <odom_topic>/model/my_robot/odometry</odom_topic>
       <odom_publish_frequency>30</odom_publish_frequency>
+      <frame_id>my_robot/odom</frame_id>
+      <child_frame_id>my_robot/base_link</child_frame_id>
+    </plugin>
+  </gazebo>
+  <gazebo>
+    <plugin filename="gz-sim-sensors-system" name="gz::sim::systems::Sensors">
+      <render_engine>ogre2</render_engine>
     </plugin>
   </gazebo>
