Commit message: feat:添加了导航内容

File: src/my_robot/urdf/my_robot.urdf.xacro (robot description, xacro)
@@ -9,5 +9,5 @@
   <xacro:property name="wheel_radius" value="0.05" />
   <xacro:property name="wheel_length" value="0.04" />
-  <xacro:property name="caster_radius" value="0.02" />
+  <xacro:property name="caster_radius" value="0.025" />
   <xacro:property name="caster_length" value="0.02" />
   <material name="body_color">
@@ -91,6 +91,6 @@
   <xacro:drive_wheel name="right_wheel" y="-0.12"/>
   <!-- Caster轮 -->
-  <xacro:caster_wheel name="front_caster" x="0.15" y="0" z="-0.07"/>
-  <xacro:caster_wheel name="rear_caster" x="-0.15" y="0" z="-0.07"/>
+  <xacro:caster_wheel name="front_caster" x="0.15" y="0" z="-0.075"/>
+  <xacro:caster_wheel name="rear_caster" x="-0.15" y="0" z="-0.075"/>
   <gazebo>
     <plugin

Commit message: Release:Slam and Navgigation in Jazzy

File: src/my_robot/urdf/my_robot.urdf.xacro (robot description, xacro)
@@ -62,17 +62,9 @@
     <link name="${name}">
       <visual>
-        <geometry><cylinder radius="${caster_radius}" length="${caster_length}"/></geometry>
+        <geometry><sphere radius="${caster_radius}"/></geometry>
         <material name="wheel_color"/>
       </visual>
       <collision>
-        <geometry><cylinder radius="${caster_radius}" length="${caster_length}"/></geometry>
-        <surface>
-          <friction>
-            <ode>
-              <mu1>0.1</mu1>
-              <mu2>0.1</mu2>
-            </ode>
-          </friction>
-        </surface>
+        <geometry><sphere radius="${caster_radius}"/></geometry>
       </collision>
       <inertial>
@@ -81,9 +73,14 @@
       </inertial>
     </link>
-    <joint name="${name}_joint" type="continuous">
+    <joint name="${name}_joint" type="fixed">
       <parent link="base_link"/>
       <child link="${name}"/>
-      <origin xyz="${x} ${y} ${z}" rpy="1.5708 0 0"/>
+      <origin xyz="${x} ${y} ${z}" rpy="0 0 0"/>
     </joint>
+    <gazebo reference="${name}">
+      <mu1>0.0</mu1>
+      <mu2>0.0</mu2>
+      <kp>1000000.0</kp> <kd>100.0</kd>     <material>Gazebo/Black</material>
+    </gazebo>
   </xacro:macro>
   <!-- 驱动轮 -->
